Commit message: Feat: add sensor plugins to robot follower package

File: robot_follower/urdf/robot_follower.xacro (robot description, xacro)
@@ -100,5 +100,5 @@
   <!-- Caster wheel definition (joints and links) -->
   <joint name="caster_base_joint" type="continuous">
-    <origin xyz="-0.104 0 0.015" rpy="0 0 ${PI}" />
+    <origin xyz="-0.104 0 0.025" rpy="0 0 ${PI}" />
     <parent link="base_link" />
     <child link="caster_base_link" />
@@ -143,3 +143,54 @@
     </inertial>
   </link>
+  <!-- ************************ SENSORS FRAME DEFINITION ************************ -->
+  <!-- IMU -->
+  <joint name="imu_joint" type="fixed">
+    <parent link="base_link"/>
+    <child link="imu_link"/>
+    <origin xyz="0 0 0" rpy="0 0 0"/>
+  </joint>
+  <link name="imu_link"/>
+  <!-- LIDAR -->
+  <joint name="lidar_joint" type="fixed">
+    <parent link="base_link"/>
+    <child link="lidar_link"/>
+    <origin xyz="-0.04 0 0.04" rpy="0 0 0"/>
+  </joint>
+  <link name="lidar_link">
+    <visual>
+      <origin xyz="-0.0275 -0.0275 0" rpy="0 0 0"/>
+      <geometry>
+        <mesh filename="package://${package_name}/meshes/Lidar_pacecat.stl" scale="0.001 0.001 0.001" />
+      </geometry>
+    </visual>
+  </link>
+  <!-- CAMERA -->
+  <joint name="camera_joint" type="fixed">
+    <origin xyz="0.04 0 0.055" rpy="0 0 0"/>
+    <parent link="base_link"/>
+    <child link="camera_frame"/>
+  </joint>
+  <link name="camera_frame">
+    <visual>
+      <origin xyz="0 0 0" rpy="0 0 0"/>
+      <geometry>
+        <box size="0.02 0.07 0.03"/>
+      </geometry>
+    </visual>
+    <!-- Since the camera is a sensor, collision and inertial tags are optional -->
+  </link>
+  <!-- SONAR -->
+  <joint name="sonar_joint" type="fixed">
+    <origin xyz="0.04 0 0.015" rpy="0 0 0"/>
+    <parent link="base_link"/>
+    <child link="sonar_link"/>
+  </joint>
+  <link name="sonar_link">
+    <visual>
+      <origin xyz="0 -0.025 0" rpy="${PI/2} 0 ${PI/2}"/>
+      <geometry>
+        <mesh filename="package://${package_name}/meshes/Sonar_hcsr04.stl" scale="0.001 0.001 0.001" />
+      </geometry>
+    </visual>
+  </link>
 </robot>

File: robot_follower/urdf/robot_follower_gz.xacro (robot description, xacro)
@@ -2,4 +2,7 @@
 <robot xmlns:xacro="http://ros.org/wiki/xacro">
 <!-- http://wiki.ros.org/simulator_gazebo/Tutorials/ListOfMaterials -->
+  <xacro:arg name="laser_visual"  default="false"/> <!-- With true, blue rays are shown in Gazebo-->
+  <xacro:arg name="camera_visual" default="false"/> <!-- With true, what the camera sees is shown in Gazebo-->
+  <xacro:arg name="sonar_visual"  default="false"/> <!-- With true, blue triangles are shown in Gazebo-->
   <xacro:arg name="base_color"    default="Blue"/>
   <!-- Custom color (for RViz) -->
@@ -87,3 +90,191 @@
     </plugin>
   </gazebo>
+  <!-- ******************** SENSORS PLUGINS ******************** -->
+  <!-- IMU -->
+  <gazebo reference="imu_link">
+    <sensor name="imu" type="imu">
+      <visualize>true</visualize>
+      <always_on>true</always_on>
+      <update_rate>30</update_rate>
+      <plugin name="imu_plugin" filename="libgazebo_ros_imu_sensor.so">
+        <ros>
+          <remapping>~/out:=imu</remapping>
+        </ros>
+        <initial_orientation_as_reference>false</initial_orientation_as_reference>
+      </plugin>
+      <imu>
+     	<angular_velocity>
+     	  <x>
+     	    <noise type="gaussian">
+              <mean>0.0</mean>
+              <stddev>2e-4</stddev>
+              <bias_mean>0.0000075</bias_mean>
+              <bias_stddev>0.0000008</bias_stddev>
+            </noise>
+          </x>
+          <y>
+            <noise type="gaussian">
+              <mean>0.0</mean>
+              <stddev>2e-4</stddev>
+              <bias_mean>0.0000075</bias_mean>
+              <bias_stddev>0.0000008</bias_stddev>
+            </noise>
+          </y>
+          <z>
+            <noise type="gaussian">
+              <mean>0.0</mean>
+              <stddev>2e-4</stddev>
+              <bias_mean>0.0000075</bias_mean>
+              <bias_stddev>0.0000008</bias_stddev>
+            </noise>
+          </z>
+        </angular_velocity>
+        <linear_acceleration>
+          <x>
+            <noise type="gaussian">
+              <mean>0.0</mean>
+              <stddev>1.7e-2</stddev>
+              <bias_mean>0.1</bias_mean>
+              <bias_stddev>0.001</bias_stddev>
+            </noise>
+          </x>
+          <y>
+            <noise type="gaussian">
+              <mean>0.0</mean>
+              <stddev>1.7e-2</stddev>
+              <bias_mean>0.1</bias_mean>
+              <bias_stddev>0.001</bias_stddev>
+            </noise>
+          </y>
+          <z>
+            <noise type="gaussian">
+              <mean>0.0</mean>
+              <stddev>1.7e-2</stddev>
+              <bias_mean>0.1</bias_mean>
+              <bias_stddev>0.001</bias_stddev>
+            </noise>
+          </z>
+        </linear_acceleration>
+      </imu>
+    </sensor>
+  </gazebo>
+  <!-- LIDAR -->
+  <gazebo reference="lidar_link">
+    <material>Gazebo/Black</material>
+    <sensor type="ray" name="lidar">
+      <pose>0 0 0 0 0 0</pose>
+      <visualize>$(arg laser_visual)</visualize>
+      <always_on>true</always_on>
+      <update_rate>15</update_rate>
+      <ray>
+        <scan>
+          <horizontal>
+            <samples>360</samples>
+            <resolution>1</resolution>
+            <min_angle>${-PI}</min_angle>
+            <max_angle>${PI}</max_angle>
+          </horizontal>
+        </scan>
+        <range>
+          <min>0.15</min>
+          <max>1.5</max>
+          <resolution>0.017453</resolution>
+        </range>
+        <noise>
+          <type>gaussian</type>
+          <mean>0.0</mean>
+          <stddev>0.01</stddev>
+        </noise>
+      </ray>
+      <plugin name="laser_plugin" filename="libgazebo_ros_ray_sensor.so">
+        <ros>
+            <remapping>~/out:=scan</remapping>
+        </ros>
+        <output_type>sensor_msgs/LaserScan</output_type>
+        <frame_name>lidar_link</frame_name>
+      </plugin>
+    </sensor>
+  </gazebo>
+  <!-- MONOCULAR CAMERA -->
+  <gazebo reference="camera_frame">
+    <material>Gazebo/Orange</material>
+    <sensor type="camera" name="camera">
+      <always_on>true</always_on>
+      <update_rate>30.0</update_rate>
+      <visualize>$(arg camera_visual)</visualize>
+      <camera>
+        <horizontal_fov>1.085595</horizontal_fov>
+        <image>
+          <width>640</width>
+          <height>480</height>
+          <format>R8G8B8</format>
+        </image>
+        <clip>
+          <near>0.05</near>
+          <far>8.0</far>
+        </clip>
+        <distortion>
+         <k1>0.0</k1>
+         <k2>0.0</k2>
+         <k3>0.0</k3>
+         <p1>0.0</p1>
+         <p2>0.0</p2>
+         <center>0.5 0.5</center>
+       </distortion>
+      </camera>
+        <plugin name="camera_plugin" filename="libgazebo_ros_camera.so">
+            <ros>
+                <!--namespace>/</namespace-->
+                <remapping>~/image_raw:=image_raw</remapping>
+                <remapping>~/camera_info:=camera_info</remapping>
+            </ros>
+            <camera_name>camera</camera_name>
+            <frame_name>camera_frame</frame_name>
+            <hack_baseline>0.2</hack_baseline>
+        </plugin>
+    </sensor>
+  </gazebo>
+  <!-- SONAR -->
+  <gazebo reference="sonar_link">
+    <material>Gazebo/Grey</material>
+    <sensor type="ray" name="sonar_sensor">
+      <pose>0 0 0 0 0 0</pose>
+      <visualize>$(arg sonar_visual)</visualize>
+      <update_rate>30</update_rate>
+      <ray>
+        <scan>
+          <horizontal>
+            <samples>2</samples>
+            <resolution>1</resolution>
+            <min_angle>-25</min_angle>
+            <max_angle>25</max_angle>
+          </horizontal>
+          <vertical>
+            <samples>1</samples>
+            <resolution>1</resolution>
+            <min_angle>0</min_angle>
+            <max_angle>25</max_angle>
+          </vertical>
+        </scan>
+        <range>
+          <min>0.04</min>
+          <max>0.9</max>
+          <resolution>0.01</resolution>
+        </range>
+        <noise>
+          <type>gaussian</type>
+          <mean>0.0</mean>
+          <stddev>0.01</stddev>
+        </noise>
+      </ray>
+      <plugin filename="libgazebo_ros_ray_sensor.so" name="sonar_plugin">
+        <ros>
+          <remapping>~/out:=sonar</remapping>
+        </ros>
+        <output_type>sensor_msgs/Range</output_type>
+        <radiation_type>ultrasound</radiation_type> <!-- infrared=1, ultrasound=0 -->
+        <frame_name>sonar_link</frame_name>
+      </plugin>
+    </sensor>
+  </gazebo>
 </robot>
